Commit message: update urdf model

File: models/iris_gimbal/iris_gimbal.urdf (robot description, URDF)
Before this commit: robot iris_gimbal, 12 links, 11 joints
Links:
- link iris_gimbal__base_link: geometry collision box size=0.47 0.47 0.11; visual mesh filename=package://mavlink_sitl_gazebo/models/rotors_description/mes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 scale=1 1 1
- link iris_gimbal__cgo3_camera_link: geometry collision sphere radius=0.035; visual mesh filename=package://mavlink_sitl_gazebo/models/typhoon_h480/meshes/cg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 scale=0.001 0.001 0.001
- link iris_gimbal__cgo3_horizontal_arm_link: geometry visual mesh filename=package://mavlink_sitl_gazebo/models/typhoon_h480/meshes/cg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 scale=0.001 0.001 0.001
- link iris_gimbal__cgo3_mount_link: geometry visual mesh filename=package://mavlink_sitl_gazebo/models/typhoon_h480/meshes/cg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 scale=0.001 0.001 0.001
- link iris_gimbal__cgo3_vertical_arm_link: geometry visual mesh filename=package://mavlink_sitl_gazebo/models/typhoon_h480/meshes/cg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 scale=0.001 0.001 0.001
- link iris_gimbal__left_leg: geometry collision box size=0.024418 0.024418 0.3; collision cylinder length=0.176893 radius=0.00914984
- link iris_gimbal__right_leg: geometry collision box size=0.024418 0.024418 0.3; collision cylinder length=0.176893 radius=0.00914984
- link iris_gimbal__rotor_0: geometry collision cylinder length=0.005 radius=0.128; visual mesh filename=package://mavlink_sitl_gazebo/models/rotors_description/mes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 scale=1 1 1
- link iris_gimbal__rotor_1: geometry collision cylinder length=0.005 radius=0.128; visual mesh filename=package://mavlink_sitl_gazebo/models/rotors_description/mes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 scale=1 1 1
- link iris_gimbal__rotor_2: geometry collision cylinder length=0.005 radius=0.128; visual mesh filename=package://mavlink_sitl_gazebo/models/rotors_description/mes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 scale=1 1 1
- link iris_gimbal__rotor_3: geometry collision cylinder length=0.005 radius=0.128; visual mesh filename=package://mavlink_sitl_gazebo/models/rotors_description/mes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 scale=1 1 1

Commit message: .

File: models/iris_gimbal/iris_gimbal.urdf (robot description, URDF)
Before this commit: robot iris_gimbal, 12 links, 11 joints
Links:
- removed link iris_gimbal__/imu_link
- removed link iris_gimbal__base_link
- removed link iris_gimbal__cgo3_camera_link
- removed link iris_gimbal__cgo3_horizontal_arm_link
- removed link iris_gimbal__cgo3_mount_link
- removed link iris_gimbal__cgo3_vertical_arm_link
- removed link iris_gimbal__left_leg
- removed link iris_gimbal__right_leg
- removed link iris_gimbal__rotor_0
- removed link iris_gimbal__rotor_1
- removed link iris_gimbal__rotor_2
- removed link iris_gimbal__rotor_3
- added link /imu_link, mass 0.015
- added link base_link, mass 1.5; collision box size=0.47 0.47 0.11; visual mesh filename=package://mavlink_sitl_gazebo/models/rotors_description/mes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 scale=1 1 1
- added link cgo3_camera_link, mass 0.11; collision sphere radius=0.035; visual mesh filename=package://mavlink_sitl_gazebo/models/typhoon_h480/meshes/cg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 scale=0.001 0.001 0.001
- added link cgo3_horizontal_arm_link, mass 0.11; visual mesh filename=package://mavlink_sitl_gazebo/models/typhoon_h480/meshes/cg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 scale=0.001 0.001 0.001
- added link cgo3_mount_link, mass 0.11; visual mesh filename=package://mavlink_sitl_gazebo/models/typhoon_h480/meshes/cg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 scale=0.001 0.001 0.001
- added link cgo3_vertical_arm_link, mass 0.11; visual mesh filename=package://mavlink_sitl_gazebo/models/typhoon_h480/meshes/cg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 scale=0.001 0.001 0.001
- added link left_leg, mass 0.1; collision box size=0.024418 0.024418 0.3; collision cylinder length=0.176893 radius=0.00914984
- added link right_leg, mass 0.1; collision box size=0.024418 0.024418 0.3; collision cylinder length=0.176893 radius=0.00914984
- added link rotor_0, mass 0.005; collision cylinder length=0.005 radius=0.128; visual mesh filename=package://mavlink_sitl_gazebo/models/rotors_description/mes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 scale=1 1 1
- added link rotor_1, mass 0.005; collision cylinder length=0.005 radius=0.128; visual mesh filename=package://mavlink_sitl_gazebo/models/rotors_description/mes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 scale=1 1 1
- added link rotor_2, mass 0.005; collision cylinder length=0.005 radius=0.128; visual mesh filename=package://mavlink_sitl_gazebo/models/rotors_description/mes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 scale=1 1 1
- added link rotor_3, mass 0.005; collision cylinder length=0.005 radius=0.128; visual mesh filename=package://mavlink_sitl_gazebo/models/rotors_description/mes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 scale=1 1 1
Joints:
- removed joint iris_gimbal__/imu_joint
- removed joint iris_gimbal__cgo3_camera_joint
- removed joint iris_gimbal__cgo3_horizontal_arm_joint
- removed joint iris_gimbal__cgo3_mount_joint
- removed joint iris_gimbal__cgo3_vertical_arm_joint
- removed joint iris_gimbal__left_leg_joint
- removed joint iris_gimbal__right_leg_joint
- removed joint iris_gimbal__rotor_0_joint
- removed joint iris_gimbal__rotor_1_joint
- removed joint iris_gimbal__rotor_2_joint
- removed joint iris_gimbal__rotor_3_joint
- added joint /imu_joint: type fixed, parent base_link, child /imu_link, origin xyz=0   0   0 rpy=0 0 0, axis 1 0 0, limit lower=0.0 upper=0.0 effort=0.0 velocity=0.0
- added joint cgo3_camera_joint: type revolute, parent cgo3_horizontal_arm_link, child cgo3_camera_link, origin xyz=-0.067  0.03   0 rpy=0 0 0, axis 0 1 0, limit lower=-315.0 upper=315.0 effort=100.0 velocity=-1.0
- added joint cgo3_horizontal_arm_joint: type revolute, parent cgo3_vertical_arm_link, child cgo3_horizontal_arm_link, origin xyz=0.052  0    -0.062 rpy=0 0 0, axis 1 0 0, limit lower=-785398.0 upper=785398.0 effort=100.0 velocity=-1.0
- added joint cgo3_mount_joint: type fixed, parent base_link, child cgo3_mount_link, origin xyz=0      0      0.026 rpy=0      0      3.14159, axis 0 0 1, limit lower=0.0 upper=0.0 effort=100.0 velocity=-1.0
- added joint cgo3_vertical_arm_joint: type revolute, parent cgo3_mount_link, child cgo3_vertical_arm_link, origin xyz=-0.026  0    -0.1 rpy=0 0 0, axis 0 0 1, limit lower=-1e+16 upper=1e+16 effort=100.0 velocity=-1.0
- added joint left_leg_joint: type revolute, parent base_link, child left_leg, origin xyz=0.00038 -0.04052  0.229 rpy=-0.00021 -0.00233  0.0003, axis -9.9999e-01  3.0000e-04  2.3300e-03, limit lower=0.0 upper=1.0 effort=100.0 velocity=-1.0
- added joint right_leg_joint: type revolute, parent base_link, child right_leg, origin xyz=1.2000e-04 4.0570e-02 2.2904e-01 rpy=0.00119 0.00126 0.0018, axis 0.99999 -0.0018   0.00126, limit lower=0.0 upper=1.0 effort=100.0 velocity=-1.0
- added joint rotor_0_joint: type revolute, parent base_link, child rotor_0, origin xyz=0.1295  -0.2188   0.026 rpy=0 0 0, axis 0 0 1, limit lower=-1e+16 upper=1e+16 effort=0.0 velocity=0.0
- added joint rotor_1_joint: type revolute, parent base_link, child rotor_1, origin xyz=-0.1338   0.2065   0.026 rpy=0 0 0, axis 0 0 1, limit lower=-1e+16 upper=1e+16 effort=0.0 velocity=0.0
- added joint rotor_2_joint: type revolute, parent base_link, child rotor_2, origin xyz=0.1257  0.2225  0.026 rpy=0 0 0, axis 0 0 1, limit lower=-1e+16 upper=1e+16 effort=0.0 velocity=0.0
- added joint rotor_3_joint: type revolute, parent base_link, child rotor_3, origin xyz=-0.1375  -0.203    0.026 rpy=0 0 0, axis 0 0 1, limit lower=-1e+16 upper=1e+16 effort=0.0 velocity=0.0

Commit message: update

File: models/iris_gimbal/iris_gimbal.urdf (robot description, URDF)
Before this commit: robot iris_gimbal, 12 links, 11 joints
Links:
- link base_link: geometry collision box size=0.47 0.47 0.11; visual mesh filename=package://offbnode/models/iris_gimbal/meshes/iris.stl scale=1 1 1
- link cgo3_camera_link: geometry collision sphere radius=0.035; visual mesh filename=package://offbnode/models/iris_gimbal/meshes/cgo3_camera_re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 scale=0.001 0.001 0.001
- link cgo3_horizontal_arm_link: geometry visual mesh filename=package://offbnode/models/iris_gimbal/meshes/cgo3_horizonta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 scale=0.001 0.001 0.001
- link cgo3_mount_link: geometry visual mesh filename=package://offbnode/models/iris_gimbal/meshes/cgo3_mount_rem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 scale=0.001 0.001 0.001
- link cgo3_vertical_arm_link: geometry visual mesh filename=package://offbnode/models/iris_gimbal/meshes/cgo3_vertical_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 scale=0.001 0.001 0.001
- link left_leg: geometry collision box size=0.024418 0.024418 0.3; collision cylinder length=0.176893 radius=0.00914984
- link right_leg: geometry collision box size=0.024418 0.024418 0.3; collision cylinder length=0.176893 radius=0.00914984
- link rotor_0: geometry collision cylinder length=0.005 radius=0.128; visual mesh filename=package://offbnode/models/iris_gimbal/meshes/iris_prop_ccw.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 scale=1 1 1
- link rotor_1: geometry collision cylinder length=0.005 radius=0.128; visual mesh filename=package://offbnode/models/iris_gimbal/meshes/iris_prop_ccw.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 scale=1 1 1
- link rotor_2: geometry collision cylinder length=0.005 radius=0.128; visual mesh filename=package://offbnode/models/iris_gimbal/meshes/iris_prop_cw.d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 scale=1 1 1
- link rotor_3: geometry collision cylinder length=0.005 radius=0.128; visual mesh filename=package://offbnode/models/iris_gimbal/meshes/iris_prop_cw.d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 scale=1 1 1
Joints:
- joint left_leg_joint: origin xyz=0.00038 -0.04052  0.229 rpy=-0.00021 -0.00233  0.0003 -> xyz=0.00038 -0.04052  -0.031 rpy=-0.00021 -0.00233  0.0003
- joint right_leg_joint: origin xyz=1.2000e-04 4.0570e-02 2.2904e-01 rpy=0.00119 0.00126 0.0018 -> xyz=1.2000e-04 4.0570e-02 -0.031 rpy=0.00119 0.00126 0.0018

Commit message: update

File: models/iris_gimbal/iris_gimbal.urdf (robot description, URDF)
Before this commit: robot iris_gimbal, 12 links, 11 joints
Links:
- added link cgo3_camera_optical_link, mass 1e-9
Joints:
- added joint cgo3_camera_optical_joint: type fixed, parent cgo3_camera_link, child cgo3_camera_optical_link, origin xyz=0.041  0    -0.136 rpy=0 -1.5707963 0, axis 1 0 0, limit lower=0 upper=0 effort=0 velocity=0

Commit message: update sdf con joint de camara

File: models/iris_gimbal/iris_gimbal.urdf (robot description, URDF)
Before this commit: robot iris_gimbal, 13 links, 12 joints
Joints:
- joint cgo3_camera_optical_joint: axis 1 0 0 -> 0 0 1; origin xyz=0.041  0    -0.136 rpy=0 -1.5707963 0 -> xyz=0   -0.03  0 rpy=0      -1.57079 -3.14159

Commit message: Update iris_gimbal.urdf

File: models/iris_gimbal/iris_gimbal.urdf (robot description, URDF)
Before this commit: robot iris_gimbal, 13 links, 12 joints
Links:
- link cgo3_camera_link: mass 0.11 -> 0.02
- link cgo3_horizontal_arm_link: mass 0.11 -> 0.01
- link cgo3_mount_link: mass 0.11 -> 0.01
- link cgo3_vertical_arm_link: mass 0.11 -> 0.01
Joints:
- joint /imu_joint: origin xyz=0   0   0 rpy=0 0 0 -> xyz=0 0 0 rpy=0 0 0
- joint cgo3_camera_joint: limit lower=-315.0 upper=315.0 effort=100.0 velocity=-1.0 -> lower=-31500.0 upper=31500.0 effort=1.0 velocity=-1.0
- joint cgo3_camera_optical_joint: limit lower=0 upper=0 effort=0 velocity=0 -> lower=0.0 upper=0.0 effort=0.0 velocity=0.0; origin xyz=0   -0.03  0 rpy=0      -1.57079 -3.14159 -> xyz=0   -0.03  0 rpy=0       1.57079 -3.14159
- joint cgo3_horizontal_arm_joint: limit lower=-785398.0 upper=785398.0 effort=100.0 velocity=-1.0 -> lower=-785398.0 upper=785398.0 effort=1.0 velocity=1.0
- joint cgo3_mount_joint: limit lower=0.0 upper=0.0 effort=100.0 velocity=-1.0 -> lower=0.0 upper=0.0 effort=0.0 velocity=-1.0; origin xyz=0      0      0.026 rpy=0      0      3.14159 -> xyz=-0.026  0     0.026 rpy=0      0      3.14159
- joint cgo3_vertical_arm_joint: limit lower=-1e+16 upper=1e+16 effort=100.0 velocity=-1.0 -> lower=-1e+16 upper=1e+16 effort=1.0 velocity=-1.0
- joint left_leg_joint: origin xyz=0.00038 -0.04052  -0.031 rpy=-0.00021 -0.00233  0.0003 -> xyz=0.00038 -0.04052 -0.03099 rpy=-0.00021 -0.00233  0.0003
- joint right_leg_joint: origin xyz=1.2000e-04 4.0570e-02 -0.031 rpy=0.00119 0.00126 0.0018 -> xyz=0.00012  0.04057 -0.03095 rpy=0.00119 0.00126 0.0018
- joint rotor_0_joint: origin xyz=0.1295  -0.2188   0.026 rpy=0 0 0 -> xyz=0.1295 -0.2188  0.026 rpy=0 0 0
- joint rotor_1_joint: origin xyz=-0.1338   0.2065   0.026 rpy=0 0 0 -> xyz=-0.1338  0.2065  0.026 rpy=0 0 0
- joint rotor_2_joint: origin xyz=0.1257  0.2225  0.026 rpy=0 0 0 -> xyz=0.1257 0.2225 0.026 rpy=0 0 0
- joint rotor_3_joint: origin xyz=-0.1375  -0.203    0.026 rpy=0 0 0 -> xyz=-0.1375 -0.203   0.026 rpy=0 0 0

Commit message: Medicion de plano de terreno completa

File: models/iris_gimbal/iris_gimbal.urdf (robot description, URDF)
Before this commit: robot iris_gimbal, 13 links, 12 joints
Joints:
- joint cgo3_camera_optical_joint: origin xyz=0   -0.03  0 rpy=0       1.57079 -3.14159 -> xyz=0   -0.03  0 rpy=-1.57079  0  1.57079

Commit message: x

File: models/iris_gimbal/iris_gimbal.urdf (robot description, URDF)
Before this commit: robot iris_gimbal, 13 links, 12 joints
Links:
- link base_link: mass 1.5 -> None

Commit message: prueba

File: models/iris_gimbal/iris_gimbal.urdf (robot description, URDF)
Before this commit: robot iris_gimbal, 13 links, 12 joints
Links:
- added link iris_gimbal/cgo3_camera_optical_link, mass 1e-9
Joints:
- added joint iris_gimbal/cgo3_camera_optical_joint: type fixed, parent cgo3_camera_link, child iris_gimbal/cgo3_camera_optical_link, origin xyz=0   -0.03  0 rpy=-1.57079  0  1.57079, axis 0 0 1, limit lower=0.0 upper=0.0 effort=0.0 velocity=0.0
