Commit message: update

File: models/hitl_iris_gimbal/iris_gimbal.urdf (robot description, URDF)
Before this commit: robot iris_gimbal, 14 links, 13 joints
Links:
- removed link hitl_iris_gimbal/cgo3_camera_optical_link
- added link iris_gimbal/cgo3_camera_optical_link, mass 1e-9
- link base_link: geometry collision box size=0.47 0.47 0.11; visual mesh filename=package://offbnode/models/iris_gimbal/meshes/iris.stl scale=1 1 1
- link cgo3_camera_link: geometry collision sphere radius=0.035; visual mesh filename=package://offbnode/models/iris_gimbal/meshes/cgo3_camera_re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 scale=0.001 0.001 0.001
- link cgo3_horizontal_arm_link: geometry visual mesh filename=package://offbnode/models/iris_gimbal/meshes/cgo3_horizonta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 scale=0.001 0.001 0.001
- link cgo3_mount_link: geometry visual mesh filename=package://offbnode/models/iris_gimbal/meshes/cgo3_mount_rem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 scale=0.001 0.001 0.001
- link cgo3_vertical_arm_link: geometry visual mesh filename=package://offbnode/models/iris_gimbal/meshes/cgo3_vertical_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 scale=0.001 0.001 0.001
- link left_leg: geometry collision box size=0.024418 0.024418 0.3; collision cylinder length=0.176893 radius=0.00914984
- link right_leg: geometry collision box size=0.024418 0.024418 0.3; collision cylinder length=0.176893 radius=0.00914984
- link rotor_0: geometry collision cylinder length=0.005 radius=0.128; visual mesh filename=package://offbnode/models/iris_gimbal/meshes/iris_prop_ccw.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 scale=1 1 1
- link rotor_1: geometry collision cylinder length=0.005 radius=0.128; visual mesh filename=package://offbnode/models/iris_gimbal/meshes/iris_prop_ccw.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 scale=1 1 1
- link rotor_2: geometry collision cylinder length=0.005 radius=0.128; visual mesh filename=package://offbnode/models/iris_gimbal/meshes/iris_prop_cw.d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 scale=1 1 1
- link rotor_3: geometry collision cylinder length=0.005 radius=0.128; visual mesh filename=package://offbnode/models/iris_gimbal/meshes/iris_prop_cw.d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 scale=1 1 1
Joints:
- removed joint hitl_iris_gimbal/cgo3_camera_optical_joint
- added joint iris_gimbal/cgo3_camera_optical_joint: type fixed, parent cgo3_camera_link, child iris_gimbal/cgo3_camera_optical_link, origin xyz=0   -0.03  0 rpy=-1.57079  0  1.57079, axis 0 0 1, limit lower=0.0 upper=0.0 effort=0.0 velocity=0.0
